File: Satyrr_six_loadcell_pcb.sch (EAGLE design)
At the start: 49 parts, among them IC1 STM32G431KBU6, J2 SM02BGHSTBLFSN, J3 SM04B-GHS-TB(LF)(SN)-, J4 SM04B-GHS-TB(LF)(SN)-, J5 SM04B-GHS-TB(LF)(SN)-, J6 SM04B-GHS-TB(LF)(SN)-, J7 SM04B-GHS-TB(LF)(SN)-, J8 SM04B-GHS-TB(LF)(SN)-, J9 22057025, U1 MCP2562FD-H/MFDFN8_3X3MC_MCH-M, U2 AP7361C-33Y5-13SOT89-5_DIO-M, Y1 ECS-80-18-33-JGN-TR

Commit message: board finished, ready for design review
Parts:
- added JP1: (no value), pinhead:PINHD-2X9
- added JP2: (no value), pinhead:PINHD-2X4
Connections:
- removed net N$13: IC1.PA0
- removed net N$14: IC1.PA1
- removed net N$34: IC1.PB8-BOOT0
- removed net N$35: IC1.PB7
- removed net N$36: IC1.PB6
- removed net N$37: IC1.PB5
- removed net N$38: IC1.PB4
- removed net N$39: IC1.PB3
- removed net N$40: IC1.PA15
- new net GPIO0_SCL: IC1.PB8-BOOT0, JP1.5
- new net GPIO1_SDA: IC1.PB7, JP1.7
- new net GPIO2: IC1.PB6, JP1.9
- new net GPIO3: IC1.PB5, JP1.11
- new net GPIO4_RX: IC1.PB4, JP1.13
- new net GPIO5_TX: IC1.PB3, JP1.15
- new net GPIO6: IC1.PA15, JP1.17
- new net GPIO7_ADC1: IC1.PA0, JP1.1
- new net GPIO8_ADC2: IC1.PA1, JP1.3
- net 3V3: now also JP1.2, JP1.4, JP2.1, JP2.3
- net 5V: now also JP2.5, JP2.7
- net GND: now also JP1.10, JP1.12, JP1.14, JP1.16, JP1.18, JP1.6, JP1.8, JP2.2, JP2.4, JP2.6, JP2.8

Commit message: schemetic design review complete
Connections:
- removed net N$18: U1.STBY
- net FDCAN_RX: now also U1.RXD; no longer U1.TXD
- net FDCAN_TX: now also U1.TXD; no longer U1.RXD
- net GND: now also U1.STBY
Other:
- note added: "5v Power In Connector"
- note added: "5v to 3v Regulator"
- note added: "ADS1220 Loadcell Amplifier #2"
- note added: "Bypass Capacitors for STM32"
- note added: "CAN Connector"
- note added: "CAN Transceiver"
- note added: "Connectors"
- note added: "External Oscillator"
- note added: "Extra GPIO Pins"
- note added: "Extra Power Out Pins"
- note added: "Loadcell Connectors"
- note added: "STM32"
- note added: "STM32G431 Microcontroller"
- note added: "SWD Programming Connector"
- note added: "Supporting Devices"
- note added: "U$2"
